File: pcb/GLCD-Shield_v10.sch (EAGLE design)
At the start: 40 parts, among them Q1 16MHz, T1 N-CHN, U1 TS5204, X1 PASSER, X2 PASSER, X3 PASSER, X4 PASSER

Commit message: updated schematic and layout files
Parts:
- U1: value TS5204 -> TS5204-3V3
Changed lines of the file:
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@@
 <?xml version="1.0" encoding="utf-8"?>
 <!DOCTYPE eagle SYSTEM "eagle.dtd">
-<eagle version="6.5.0">
+<eagle version="6.6.0">
 <drawing>
 <settings>
@@
 <part name="A1" library="Arduino" deviceset="UNO" device=""/>
 <part name="GND14" library="supply1" deviceset="GND" device=""/>
-<part name="U1" library="Voltage-Reg" deviceset="TS5204" device=""/>
+<part name="U1" library="Voltage-Reg" deviceset="TS5204" device="" value="TS5204-3V3"/>
 <part name="ENC" library="Encoder-IR" deviceset="EC12E_SW" device=""/>
 <part name="LCD" library="Display" deviceset="UG12D228AA" device=""/>
