File: pcb/GLCD-Shield_v10.sch (EAGLE design)
At the start: 40 parts, among them Q1 16MHz, T1 N-CHN, U1 TS5204-3V3, X1 PASSER, X2 PASSER, X3 PASSER, X4 PASSER

Commit message: cleaned up schematics and layout
Changed lines of the file:
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@@
 <setting verticaltext="up"/>
 </settings>
-<grid distance="0.1" unitdist="inch" unit="inch" style="lines" multiple="1" display="no" altdistance="0.01" altunitdist="inch" altunit="inch"/>
+<grid distance="0.05" unitdist="inch" unit="inch" style="lines" multiple="1" display="yes" altdistance="0.025" altunitdist="inch" altunit="inch"/>
 <layers>
 <layer number="1" name="Top" color="4" fill="1" visible="no" active="no"/>
@@
 <parts>
 <part name="GND9" library="supply1" deviceset="GND" device=""/>
-<part name="FRAME1" library="frames" deviceset="A4L-LOC" device=""/>
 <part name="GND10" library="supply1" deviceset="GND" device=""/>
 <part name="+3V11" library="supply1" deviceset="+3V3" device=""/>
@@
 <part name="2" library="jumper" deviceset="SJ" device=""/>
 <part name="RST" library="jumper" deviceset="SJ" device=""/>
+<part name="FRAME1" library="we-symbol" deviceset="FRAME-A4L" device=""/>
 </parts>
 <sheets>
@@
 <wire x1="71.755" y1="137.16" x2="73.025" y2="137.16" width="0.4064" layer="94"/>
 <wire x1="132.08" y1="159.385" x2="132.08" y2="160.655" width="0.4064" layer="94"/>
-<text x="161.29" y="31.75" size="1.27" layer="95">Released under the Creative Commons Attribution Share-Alike License</text>
-<text x="161.29" y="29.21" size="1.27" layer="95">http://creativecommons.org/licenses/by-sa/4.0/</text>
-<text x="161.29" y="25.4" size="1.27" layer="95">Designed by Andreas Watterott (Watterott electronic)</text>
+<text x="162.56" y="21.59" size="1.27" layer="95">Released under the Creative Commons Attribution Share-Alike License</text>
+<text x="162.56" y="19.05" size="1.27" layer="95">http://creativecommons.org/licenses/by-sa/4.0/</text>
+<text x="162.56" y="15.24" size="1.27" layer="95">Designed by Andreas Watterott (Watterott electronic)</text>
 <text x="45.72" y="166.37" size="3.81" layer="250">Arduino</text>
 <text x="222.25" y="85.725" size="2.54" layer="250">FTDI Connector</text>
@@
 <attribute name="VALUE" x="91.44" y="6.35" size="1.778" layer="96"/>
 </instance>
-<instance part="FRAME1" gate="G$1" x="0" y="0" smashed="yes">
-<attribute name="DRAWING_NAME" x="217.17" y="15.24" size="2.54" layer="94" font="vector"/>
-<attribute name="LAST_DATE_TIME" x="217.17" y="10.16" size="2.286" layer="94" font="vector"/>
-<attribute name="SHEET" x="230.505" y="5.08" size="2.54" layer="94" font="vector"/>
-</instance>
 <instance part="GND10" gate="1" x="140.97" y="8.89" smashed="yes">
 <attribute name="VALUE" x="138.43" y="6.35" size="1.778" layer="96"/>
@@
 <attribute name="VALUE" x="80.01" y="143.51" size="1.778" layer="96"/>
 </instance>
-<instance part="X1" gate="G$1" x="166.37" y="19.05"/>
-<instance part="X2" gate="G$1" x="173.99" y="19.05"/>
-<instance part="X3" gate="G$1" x="181.61" y="19.05"/>
+<instance part="X1" gate="G$1" x="165.1" y="7.62" smashed="yes"/>
+<instance part="X2" gate="G$1" x="170.18" y="7.62" smashed="yes"/>
+<instance part="X3" gate="G$1" x="175.26" y="7.62" smashed="yes"/>
 <instance part="GND8" gate="1" x="121.92" y="55.88" smashed="yes" rot="MR90">
 <attribute name="VALUE" x="119.38" y="53.34" size="1.778" layer="96" rot="MR90"/>
@@
 <attribute name="VALUE" x="102.87" y="8.763" size="1.778" layer="96"/>
 </instance>
-<instance part="LOGO1" gate="G$1" x="201.93" y="11.43"/>
+<instance part="LOGO1" gate="G$1" x="198.12" y="7.62"/>
 <instance part="A1" gate="G$1" x="46.99" y="137.16"/>
 <instance part="GND14" gate="1" x="24.13" y="142.24" smashed="yes" rot="R270">
@@
 <attribute name="NAME" x="237.49" y="78.74" size="1.778" layer="95"/>
 </instance>
-<instance part="U$1" gate="G$1" x="201.93" y="19.05"/>
+<instance part="U$1" gate="G$1" x="208.28" y="7.62"/>
 <instance part="7" gate="1" x="72.39" y="137.16" smashed="yes">
 <attribute name="NAME" x="78.105" y="135.89" size="1.778" layer="95"/>
@@
 <attribute name="VALUE" x="69.85" y="123.19" size="1.778" layer="96"/>
 </instance>
-<instance part="X4" gate="G$1" x="189.23" y="19.05"/>
+<instance part="X4" gate="G$1" x="180.34" y="7.62" smashed="yes"/>
 <instance part="SW" gate="Q$1" x="35.56" y="16.51"/>
 <instance part="GND12" gate="1" x="48.26" y="8.89" smashed="yes" rot="R90">
@@
 <attribute name="VALUE" x="135.89" y="157.48" size="1.778" layer="96" rot="R90"/>
 </instance>
+<instance part="FRAME1" gate="G$1" x="0" y="0"/>
 </instances>
 <busses>
